Commit message: final urdf webcam

File: webcam_description/robots/webcam_project.urdf (robot description, URDF)
Before this commit: robot webcam_project, 5 links, 4 joints
Links:
- removed link servo1
- removed link servo2
- removed link w
- removed link webcam_support
- added link base, mass 124555.984375e-15; collision mesh filename=package://webcam_description/meshes/base_def_collision.stl scale=0.01 0.01 0.01; visual mesh filename=package://webcam_description/meshes/base_def.stl scale=0.01 0.01 0.01
- added link body, mass 71232.75e-15; visual mesh filename=package://webcam_description/meshes/body_def.stl scale=0.01 0.01 0.01
- added link head, mass 94819.84375e-15; collision mesh filename=package://webcam_description/meshes/head_def_collision.stl scale=0.01 0.01 0.01; visual mesh filename=package://webcam_description/meshes/head_def.stl scale=0.01 0.01 0.01
- added link world
- link webcam: mass None -> 36673.832031e-15; geometry visual mesh filename=package://webcam_description/meshes/camera_def.stl scale=0.01 0.01 0.01
Joints:
- removed joint servo1_to_servo2
- removed joint servo2_to_webcam_support
- removed joint webcam_support_to_webcam
- removed joint world_to_servo1
- added joint base_to_body: type revolute, parent base, child body, origin xyz=0 0 0.47, axis 0 0 1, limit lower=-3.1415 upper=3.1415 effort=10.0 velocity=0.5
- added joint body_to_head: type revolute, parent body, child head, origin xyz=-0.362 0 0.75 rpy=0 0 0, axis 1 0 0, limit lower=-0.9 upper=0.2 effort=10.0 velocity=0.5
- added joint head_to_webcam: type fixed, parent head, child webcam, origin xyz=0.475 -0.35 -0.005 rpy=0 0 -1.5707
- added joint world_to_base: type fixed, parent world, child base, origin xyz=0 0 0 rpy=0 0 0, axis 0 0 1
